File: Bus_switch.kicad_sch (KiCad schematic)
At the start: 15 parts, among them J3 Conn_01x04_Pin, U1 SN74CB3Q3384APW

Commit message: finished schematic
Parts:
- removed R4: 10kΩ, PCM_JLCPCB:R_0402, symbol PCM_JLCPCB-Resistors:0402,10kΩ
- removed U1: SN74CB3Q3384APW, Package_SO:TSSOP-24_4.4x7.8mm_P0.65mm, symbol 74xx:SN74CB3Q3384APW
- added R19: 10kΩ, PCM_JLCPCB:R_0402, symbol PCM_JLCPCB-Resistors:0402,10kΩ
- added U1: SN74CB3Q3245PWR, SN74CB3Q3245PWR:TSSOP-20_L6.5-W4.4-P0.65-LS6.4-BL, symbol SN74CB3Q3245PWR:SN74CB3Q3245PWR
- R7, R8: now not fitted; now left out of the parts list
Connections:
- net +3V3: now also R19.2, U1.20 (VCC)
- net Chainbus.CS: now also U1.13 (B6)
- net Chainbus.MISO: now also U1.16 (B3)
- net Chainbus.MOSI: now also U1.15 (B4)
- net Chainbus.RX: now also U1.18 (B1)
- net Chainbus.SCK: now also U1.14 (B5)
- net Chainbus.SCL: now also U1.12 (B7)
- net Chainbus.SDA: now also U1.11 (B8)
- net Chainbus.TX: now also U1.17 (B2)
- net Chainbus_In.CS: now also U1.7 (A6)
- net Chainbus_In.MISO: now also U1.4 (A3)
- net Chainbus_In.MOSI: now also U1.5 (A4)
- net Chainbus_In.RX: now also U1.2 (A1)
- net Chainbus_In.SCK: now also U1.6 (A5)
- net Chainbus_In.SCL: now also U1.8 (A7)
- net Chainbus_In.SDA: now also U1.9 (A8)
- net Chainbus_In.TX: now also U1.3 (A2)
- net GND: now also U1.10 (GND)
- net SEL1: now also R19.1, U1.19 (~{OE})
- no-connect marks 4 -> 1
Other:
- company: (none) -> MiniModucard System
- title: MMS3 Hat template small (Change Me) -> MMS3_hat_ruski_wentylator_do_pieca
