File: Interboard_connector.kicad_sch (KiCad schematic)
At the start: 2 parts, among them J1 Chainbus in, J2 Chainbus Out

Commit message: finished schematic
Other:
- company: Moducard System -> MiniModucard System
- title: MMS3 Hat template small (Change Me) -> MMS3_hat_ruski_wentylator_do_pieca
Changed lines of the file:
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@@
 	(paper "A4")
 	(title_block
-		(title "MMS3 Hat template small (Change Me)")
+		(title "MMS3_hat_ruski_wentylator_do_pieca")
 		(date "2026-02-25")
 		(rev "A")
-		(company "Moducard System")
-		(comment 1 "Made by Wojciech Szafrański")
+		(company "MiniModucard System")
+		(comment 1 "Wojciech Szafrański")
 		(comment 2 "Designed in poland")
 	)
@@
 		)
 		(instances
-			(project "MMS3_hat_templates"
+			(project "MMS3_hat_ruski_wentylator_do_pieca"
 				(path "/6596548a-44e0-46d8-8624-fd71cf4a3e17/fdb595ff-e94b-4e80-8fe7-e7d367588ab2"
 					(reference "#PWR016")
@@
 		)
 		(instances
-			(project "MMS3_hat_templates"
+			(project "MMS3_hat_ruski_wentylator_do_pieca"
 				(path "/6596548a-44e0-46d8-8624-fd71cf4a3e17/fdb595ff-e94b-4e80-8fe7-e7d367588ab2"
 					(reference "#PWR014")
@@
 		)
 		(instances
-			(project "MMS3_hat_templates"
+			(project "MMS3_hat_ruski_wentylator_do_pieca"
 				(path "/6596548a-44e0-46d8-8624-fd71cf4a3e17/fdb595ff-e94b-4e80-8fe7-e7d367588ab2"
 					(reference "#PWR023")
@@
 		)
 		(instances
-			(project "MMS3_hat_templates"
+			(project "MMS3_hat_ruski_wentylator_do_pieca"
 				(path "/6596548a-44e0-46d8-8624-fd71cf4a3e17/fdb595ff-e94b-4e80-8fe7-e7d367588ab2"
 					(reference "#PWR012")
@@
 		)
 		(instances
-			(project "MMS3_hat_templates"
+			(project "MMS3_hat_ruski_wentylator_do_pieca"
 				(path "/6596548a-44e0-46d8-8624-fd71cf4a3e17/fdb595ff-e94b-4e80-8fe7-e7d367588ab2"
 					(reference "#PWR07")
@@
 		)
 		(instances
-			(project "MMS3_hat_templates"
+			(project "MMS3_hat_ruski_wentylator_do_pieca"
 				(path "/6596548a-44e0-46d8-8624-fd71cf4a3e17/fdb595ff-e94b-4e80-8fe7-e7d367588ab2"
 					(reference "#PWR022")
@@
 		)
 		(instances
-			(project "MMS3_hat_templates"
+			(project "MMS3_hat_ruski_wentylator_do_pieca"
 				(path "/6596548a-44e0-46d8-8624-fd71cf4a3e17/fdb595ff-e94b-4e80-8fe7-e7d367588ab2"
 					(reference "#PWR04")
@@
 		)
 		(instances
-			(project "MMS3_hat_templates"
+			(project "MMS3_hat_ruski_wentylator_do_pieca"
 				(path "/6596548a-44e0-46d8-8624-fd71cf4a3e17/fdb595ff-e94b-4e80-8fe7-e7d367588ab2"
 					(reference "#PWR025")
@@
 		)
 		(instances
-			(project "MMS3_hat_templates"
+			(project "MMS3_hat_ruski_wentylator_do_pieca"
 				(path "/6596548a-44e0-46d8-8624-fd71cf4a3e17/fdb595ff-e94b-4e80-8fe7-e7d367588ab2"
 					(reference "J2")
@@
 		)
 		(instances
-			(project "MMS3_hat_templates"
+			(project "MMS3_hat_ruski_wentylator_do_pieca"
 				(path "/6596548a-44e0-46d8-8624-fd71cf4a3e17/fdb595ff-e94b-4e80-8fe7-e7d367588ab2"
 					(reference "#PWR027")
@@
 		)
 		(instances
-			(project "MMS3_hat_templates"
+			(project "MMS3_hat_ruski_wentylator_do_pieca"
 				(path "/6596548a-44e0-46d8-8624-fd71cf4a3e17/fdb595ff-e94b-4e80-8fe7-e7d367588ab2"
 					(reference "#PWR09")
@@
 		)
 		(instances
-			(project "MMS3_hat_templates"
+			(project "MMS3_hat_ruski_wentylator_do_pieca"
 				(path "/6596548a-44e0-46d8-8624-fd71cf4a3e17/fdb595ff-e94b-4e80-8fe7-e7d367588ab2"
 					(reference "J1")
@@
 		)
 		(instances
-			(project "MMS3_hat_templates"
+			(project "MMS3_hat_ruski_wentylator_do_pieca"
 				(path "/6596548a-44e0-46d8-8624-fd71cf4a3e17/fdb595ff-e94b-4e80-8fe7-e7d367588ab2"
 					(reference "#PWR017")
@@
 		)
 		(instances
-			(project "MMS3_hat_templates"
+			(project "MMS3_hat_ruski_wentylator_do_pieca"
 				(path "/6596548a-44e0-46d8-8624-fd71cf4a3e17/fdb595ff-e94b-4e80-8fe7-e7d367588ab2"
 					(reference "#PWR021")
@@
 		)
 		(instances
-			(project "MMS3_hat_templates"
+			(project "MMS3_hat_ruski_wentylator_do_pieca"
 				(path "/6596548a-44e0-46d8-8624-fd71cf4a3e17/fdb595ff-e94b-4e80-8fe7-e7d367588ab2"
 					(reference "#PWR028")
@@
 		)
 		(instances
-			(project "MMS3_hat_templates"
+			(project "MMS3_hat_ruski_wentylator_do_pieca"
 				(path "/6596548a-44e0-46d8-8624-fd71cf4a3e17/fdb595ff-e94b-4e80-8fe7-e7d367588ab2"
 					(reference "#PWR019")
@@
 		)
 		(instances
-			(project "MMS3_hat_templates"
+			(project "MMS3_hat_ruski_wentylator_do_pieca"
 				(path "/6596548a-44e0-46d8-8624-fd71cf4a3e17/fdb595ff-e94b-4e80-8fe7-e7d367588ab2"
 					(reference "#PWR029")
@@
 		)
 		(instances
-			(project "MMS3_hat_templates"
+			(project "MMS3_hat_ruski_wentylator_do_pieca"
 				(path "/6596548a-44e0-46d8-8624-fd71cf4a3e17/fdb595ff-e94b-4e80-8fe7-e7d367588ab2"
 					(reference "#PWR020")
@@
 		)
 		(instances
-			(project "MMS3_hat_templates"
+			(project "MMS3_hat_ruski_wentylator_do_pieca"
 				(path "/6596548a-44e0-46d8-8624-fd71cf4a3e17/fdb595ff-e94b-4e80-8fe7-e7d367588ab2"
 					(reference "#PWR08")
@@
 		)
 		(instances
-			(project "MMS3_hat_templates"
+			(project "MMS3_hat_ruski_wentylator_do_pieca"
 				(path "/6596548a-44e0-46d8-8624-fd71cf4a3e17/fdb595ff-e94b-4e80-8fe7-e7d367588ab2"
 					(reference "#PWR02")
@@
 		)
 		(instances
-			(project "MMS3_hat_templates"
+			(project "MMS3_hat_ruski_wentylator_do_pieca"
 				(path "/6596548a-44e0-46d8-8624-fd71cf4a3e17/fdb595ff-e94b-4e80-8fe7-e7d367588ab2"
 					(reference "#PWR011")
@@
 		)
 		(instances
-			(project "MMS3_hat_templates"
+			(project "MMS3_hat_ruski_wentylator_do_pieca"
 				(path "/6596548a-44e0-46d8-8624-fd71cf4a3e17/fdb595ff-e94b-4e80-8fe7-e7d367588ab2"
 					(reference "#PWR018")
@@
 		)
 		(instances
-			(project "MMS3_hat_templates"
+			(project "MMS3_hat_ruski_wentylator_do_pieca"
 				(path "/6596548a-44e0-46d8-8624-fd71cf4a3e17/fdb595ff-e94b-4e80-8fe7-e7d367588ab2"
 					(reference "#PWR015")
@@
 		)
 		(instances
-			(project "MMS3_hat_templates"
+			(project "MMS3_hat_ruski_wentylator_do_pieca"
 				(path "/6596548a-44e0-46d8-8624-fd71cf4a3e17/fdb595ff-e94b-4e80-8fe7-e7d367588ab2"
 					(reference "#PWR026")
@@
 		)
 		(instances
-			(project "MMS3_hat_templates"
+			(project "MMS3_hat_ruski_wentylator_do_pieca"
 				(path "/6596548a-44e0-46d8-8624-fd71cf4a3e17/fdb595ff-e94b-4e80-8fe7-e7d367588ab2"
 					(reference "#PWR05")
@@
 		)
 		(instances
-			(project "MMS3_hat_templates"
+			(project "MMS3_hat_ruski_wentylator_do_pieca"
 				(path "/6596548a-44e0-46d8-8624-fd71cf4a3e17/fdb595ff-e94b-4e80-8fe7-e7d367588ab2"
 					(reference "#PWR06")
@@
 		)
 		(instances
-			(project "MMS3_hat_templates"
+			(project "MMS3_hat_ruski_wentylator_do_pieca"
 				(path "/6596548a-44e0-46d8-8624-fd71cf4a3e17/fdb595ff-e94b-4e80-8fe7-e7d367588ab2"
 					(reference "#PWR010")
@@
 		)
 		(instances
-			(project "MMS3_hat_templates"
+			(project "MMS3_hat_ruski_wentylator_do_pieca"
 				(path "/6596548a-44e0-46d8-8624-fd71cf4a3e17/fdb595ff-e94b-4e80-8fe7-e7d367588ab2"
 					(reference "#PWR024")
@@
 		)
 		(instances
-			(project "MMS3_hat_templates"
+			(project "MMS3_hat_ruski_wentylator_do_pieca"
 				(path "/6596548a-44e0-46d8-8624-fd71cf4a3e17/fdb595ff-e94b-4e80-8fe7-e7d367588ab2"
 					(reference "#PWR03")
@@
 		)
 		(instances
-			(project "MMS3_hat_templates"
+			(project "MMS3_hat_ruski_wentylator_do_pieca"
 				(path "/6596548a-44e0-46d8-8624-fd71cf4a3e17/fdb595ff-e94b-4e80-8fe7-e7d367588ab2"
 					(reference "#PWR013")

Commit message: commit before removing all the diodes :"
Parts:
- J1, J2: KiLib_Generator (none) -> connector/pin_header_socket
Changed lines of the file:
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@@
+			)
+		)
+		(property "KiLib_Generator" "connector/pin_header_socket"
+			(at 176.53 58.42 0)
+			(hide yes)
+			(show_name no)
+			(do_not_autoplace no)
+			(effects
+				(font
+					(size 1.27 1.27)
+				)
 			)
 		)
@@
 			(hide yes)
 			(show_name no)
+			(do_not_autoplace no)
+			(effects
+				(font
+					(size 1.27 1.27)
+				)
+			)
+		)
+		(property "KiLib_Generator" "connector/pin_header_socket"
+			(at 100.33 58.42 0)
+			(hide yes)
+			(show_name no)
