File: Power_Connector.kicad_sch (KiCad schematic)
At the start: 3 parts, among them J4 AMASS XT60 Male, J5 AMASS XT60 Female

Commit message: finished schematic
Parts:
- removed D4: SS510C, SS510C:SMC_L7.1-W6.2-LS8.1-RD, symbol SS510C:SS510C
- added D1: M7, PCM_JLCPCB:D_SMA, symbol PCM_JLCPCB-Diodes:General,M7
Connections:
- net Vin renamed VIN_BRD
- net VIN_BRD: now also D1.2
- new net VIN_Chainbus: D1.1
Other:
- note removed: "If you remove this, add direct connection betwen Vin and BRD_VIN"
- company: (none) -> MiniModucard System
- title: MMS3 Hat template small (Change Me) -> MMS3_hat_ruski_wentylator_do_pieca
