File: Hardware/MMS3_hat_ruski_wentylator_do_pieca.kicad_pcb (KiCad board)
At the start: 2 copper layers, 100 x 50 mm, 72 parts, among them J1 Chainbus in, J2 Chainbus Out, J3 Conn_01x04_Pin, J4 AMASS XT60 Male, J5 AMASS XT60 Female, J6 Conn_01x04_Socket, J7 Program, J9 Conn_01x06_Socket, Q1 PMOS, Q10 AO3401A, Q11 MMBT5401 200-300, Q12 MMBT5551 200-300, Q9 MMBT5551 200-300, U1 SN74CB3Q3245PWR, U2 M24C64, U3 XL6019E1, U4 AMS1117, U5 CH32V003FxPx, U6 MCP4161-502E/SN, X2 X322525MOB4SI

Commit message: added more readme
Parts:
- J7: footprint Connector_PinHeader_2.54mm:PinHeader_1x03_P2.54mm_Vertical -> Connector_JST:JST_XH_B3B-XH-A_1x03_P2.50mm_Vertical
- moved J7 1.94 mm to (162.6, 110.0), turned to 180 degrees
Connections:
- J1 pad 25: unconnected-(J1-Pin_25-Pad25) -> /Interboard_connector/R1
- J1 pad 27: unconnected-(J1-Pin_27-Pad27) -> /Interboard_connector/R2
- J2 pad 25: unconnected-(J2-Pin_25-Pad25) -> /Interboard_connector/R1
- J2 pad 27: unconnected-(J2-Pin_27-Pad27) -> /Interboard_connector/R2
- U5 pad 11: /Bus_switch/Chainbus.SCL -> /Bus_switch/Chainbus.SDA
- U5 pad 12: /Bus_switch/Chainbus.SDA -> /Bus_switch/Chainbus.SCL
Routing:
- net /Interboard_connector/R1: track 0.00 -> 3.51 mm, vias 0 -> 1
- net /Interboard_connector/R2: track 0.00 -> 2.89 mm, vias 0 -> 1
- net /CH32V003/SWIO: track 10.3 -> 12.0 mm
- net +3V3: track 194.4 -> 195.2 mm
- net /Bus_switch/Chainbus.SCL: track 55.9 -> 56.6 mm
- net /Bus_switch/Chainbus.SDA: track 54.4 -> 54.3 mm, vias 2 -> 3
